Commit message: Update camera joint origin position
Adjusted the camera joint origin position for better alignment.

File: play_ground/fred/auracle/description/camera.xacro (robot description, xacro)
@@ -4,5 +4,5 @@
         <parent link="chassis"/>
         <child link="camera_link"/>
-        <origin xyz="0.25 0 0.045" rpy="0 0 0"/>
+        <origin xyz="0.30 0 0.015" rpy="0 0 0"/>
     </joint>
     <link name="camera_link">
