Commit message: Add Differential to the Auracle bot

File: play_ground/fred/auracle/description/robot_core.xacro (robot description, xacro)
@@ -9,6 +9,7 @@
     <xacro:property name="rocker_width" value="0.02"/>
     <xacro:property name="rocker_height" value="0.2"/>
+     <xacro:property name="rocker_mass" value="0.2"/>
     <xacro:property name="tilted_link" value="0.1"/>
-    <xacro:property name="rocker_mass" value="0.5"/>
+    <xacro:property name="tilted_mass" value="0.5"/>
     <xacro:property name="wheel_radius" value="0.033"/>
     <xacro:property name="wheel_thickness" value="0.026"/>
@@ -39,5 +40,5 @@
         <parent link="base_link"/>
         <child link="chassis"/>
-        <origin xyz="0 0 0"/>
+        <origin xyz="0 0 0.104"/>
     </joint>
     <link name="chassis">
@@ -50,5 +51,5 @@
         </visual>
         <collision>
-            <origin xyz="${chassis_length/2} 0 ${chassis_height/2}"/>
+            <origin xyz="${chassis_length/2} 0 0"/>
             <geometry>
                 <box size="${chassis_length} ${chassis_width} ${chassis_height}"/>
@@ -62,9 +63,33 @@
         <material>Gazebo/Orange</material>
     </gazebo>
- <!-- LEFT WHEEL ROCKER LINK -->
-    <joint name="left_wheel_rocker_joint" type="continuous">
-        <parent link="base_link"/>
+ <!-- DIFFERENTIAL LINK -->
+    <joint name="differential_link" type="continuous">
+        <parent link="chassis"/>
+        <child link="differential_link"/>
+        <origin xyz="${chassis_length/2} 0 ${chassis_height+0.04}" rpy="0 0 0" />
+    </joint>
+    <link name="differential_link">
+        <visual>
+            <origin xyz="0 0 0" rpy="0 0 ${-pi/2}"/>
+            <geometry>
+                <box size="${chassis_width+2*rocker_width} ${rocker_width} 0.025"/>
+            </geometry>
+            <material name="blue"/>
+        </visual>
+        <collision>
+            <origin xyz="0 0 0" rpy="0 0 ${-pi/2}"/>
+            <geometry>
+                <box size="${chassis_width+2*rocker_width} ${rocker_width} 0.025"/>
+            </geometry>
+        </collision>
+        <xacro:inertial_box mass="${tilted_mass}" x="${tilted_link}" y="${rocker_width}" z="${rocker_height}">
+            <origin xyz="${rocker_length/2} 0 ${rocker_height/2}" rpy="0 0 0"/>
+        </xacro:inertial_box>
+    </link>
+    !-- LEFT WHEEL ROCKER LINK -->
+    <joint name="left_wheel_rocker_joint" type="fixed">
+        <parent link="differential_link"/>
         <child link="left_rocker"/>
-        <origin xyz="${chassis_length/2} ${chassis_width/2+rocker_width/2} 0" rpy="0 0 ${pi/2}" />
+        <origin xyz="0 ${chassis_width/2+rocker_width/2} ${-chassis_height-0.04}" rpy="0 0 ${pi/2}" />
     </joint>
     <link name="left_rocker">
@@ -77,10 +102,10 @@
         </visual>
         <collision>
-            <origin xyz="${rocker_length/2} 0 ${rocker_height/2}"/>
-            <geometry>
-                <box size="${rocker_length} ${rocker_width} ${rocker_height}"/>
-            </geometry>
-        </collision>
-        <xacro:inertial_box mass="${rocker_mass}" x="${rocker_length}" y="${rocker_width}" z="${rocker_height}">
+           <origin xyz="0 0 0" rpy="0 0 ${-pi/2}"/>
+            <geometry>
+                <box size="${rocker_length} ${rocker_width} 0.025"/>
+            </geometry>
+        </collision>
+        <xacro:inertial_box mass="${tilted_mass}" x="${tilted_link}" y="${rocker_width}" z="${rocker_height}">
             <origin xyz="${rocker_length/2} 0 ${rocker_height/2}" rpy="0 0 0"/>
         </xacro:inertial_box>
@@ -101,10 +126,10 @@
         </visual>
         <collision>
-            <origin xyz="${rocker_length/2} 0 ${rocker_height/2}"/>
-            <geometry>
-                <box size="${rocker_length} ${rocker_width} ${rocker_height}"/>
-            </geometry>
-        </collision>
-        <xacro:inertial_box mass="${rocker_mass}" x="${rocker_length}" y="${rocker_width}" z="${rocker_height}">
+           <origin xyz="0 0 -${tilted_link/2}" rpy="0 ${pi/2} 0"/>
+            <geometry>
+                <box size="${tilted_link} ${rocker_width} 0.025"/>
+            </geometry>
+        </collision>
+        <xacro:inertial_box mass="${tilted_mass}" x="${tilted_link}" y="${rocker_width}" z="${rocker_height}">
             <origin xyz="${rocker_length/2} 0 ${rocker_height/2}" rpy="0 0 0"/>
         </xacro:inertial_box>
@@ -125,10 +150,10 @@
         </visual>
         <collision>
-            <origin xyz="${rocker_length/2} 0 ${rocker_height/2}"/>
-            <geometry>
-                <box size="${rocker_length} ${rocker_width} ${rocker_height}"/>
-            </geometry>
-        </collision>
-        <xacro:inertial_box mass="${rocker_mass}" x="${rocker_length}" y="${rocker_width}" z="${rocker_height}">
+           <origin xyz="0 0 -${tilted_link/2}" rpy="0 ${pi/2} 0"/>
+            <geometry>
+                <box size="${tilted_link} ${rocker_width} 0.025"/>
+            </geometry>
+        </collision>
+        <xacro:inertial_box mass="${tilted_mass}" x="${tilted_link}" y="${rocker_width}" z="${rocker_height}">
             <origin xyz="${rocker_length/2} 0 ${rocker_height/2}" rpy="0 0 0"/>
         </xacro:inertial_box>
@@ -150,5 +175,5 @@
         <collision>
             <geometry>
-                <sphere radius="${wheel_radius}"/>
+                <cylinder radius="${wheel_radius}" length="${wheel_thickness}"/>
             </geometry>
         </collision>
@@ -175,11 +200,11 @@
         </visual>
         <collision>
-            <origin xyz="${rocker_length/2} 0 ${rocker_height/2}"/>
-            <geometry>
-                <box size="${rocker_length} ${rocker_width} ${rocker_height}"/>
-            </geometry>
-        </collision>
-        <xacro:inertial_box mass="${rocker_mass}" x="${rocker_length}" y="${rocker_width}" z="${rocker_height}">
-            <origin xyz="${rocker_length/2} 0 ${rocker_height/2}" rpy="0 0 0"/>
+            <origin xyz="0 0 -${tilted_link/2}" rpy="0 ${pi/2} 0"/>
+            <geometry>
+                <box size="${tilted_link} ${rocker_width} 0.025"/>
+            </geometry>
+        </collision>
+        <xacro:inertial_box mass="${tilted_mass}" x="${tilted_link}" y="${rocker_width}" z="${rocker_height}">
+            <origin xyz="${tilted_link/2} 0 ${rocker_height/2}" rpy="0 0 0"/>
         </xacro:inertial_box>
     </link>
@@ -200,5 +225,5 @@
         <collision>
             <geometry>
-                <sphere radius="${wheel_radius}"/>
+                <cylinder radius="${wheel_radius}" length="${wheel_thickness}"/>
             </geometry>
         </collision>
@@ -226,5 +251,5 @@
         <collision>
             <geometry>
-                <sphere radius="${wheel_radius}"/>
+                <cylinder radius="${wheel_radius}" length="${wheel_thickness}"/>
             </geometry>
         </collision>
@@ -238,7 +263,7 @@
     <!-- RIGHT WHEEL ROCKER LINK -->
     <joint name="right_wheel_rocker_joint" type="continuous">
-        <parent link="base_link"/>
+        <parent link="differential_link"/>
         <child link="right_rocker"/>
-        <origin xyz="${chassis_length/2} ${-chassis_width/2-rocker_width/2} 0" rpy="0 0 ${pi/2}" />
+        <origin xyz="0 ${-chassis_width/2-rocker_width/2} ${-chassis_height-0.04}" rpy="0 0 ${pi/2}" />
     </joint>
     <link name="right_rocker">
@@ -251,7 +276,7 @@
         </visual>
         <collision>
-            <origin xyz="${rocker_length/2} 0 ${rocker_height/2}"/>
-            <geometry>
-                <box size="${rocker_length} ${rocker_width} ${rocker_height}"/>
+            <origin xyz="0 0 0" rpy="0 0 ${-pi/2}"/>
+            <geometry>
+                <box size="${rocker_length} ${rocker_width} 0.025"/>
             </geometry>
         </collision>
@@ -275,7 +300,7 @@
         </visual>
         <collision>
-            <origin xyz="${rocker_length/2} 0 ${rocker_height/2}"/>
-            <geometry>
-                <box size="${rocker_length} ${rocker_width} ${rocker_height}"/>
+           <origin xyz="0 0 -${tilted_link/2}" rpy="0 ${pi/2} 0"/>
+            <geometry>
+                <box size="${tilted_link} ${rocker_width} 0.025"/>
             </geometry>
         </collision>
@@ -299,7 +324,7 @@
         </visual>
         <collision>
-            <origin xyz="${rocker_length/2} 0 ${rocker_height/2}"/>
-            <geometry>
-                <box size="${rocker_length} ${rocker_width} ${rocker_height}"/>
+           <origin xyz="0 0 -${tilted_link/2}" rpy="0 ${pi/2} 0"/>
+            <geometry>
+                <box size="${tilted_link} ${rocker_width} 0.025"/>
             </geometry>
         </collision>
@@ -324,5 +349,5 @@
         <collision>
             <geometry>
-                <sphere radius="${wheel_radius}"/>
+                <cylinder radius="${wheel_radius}" length="${wheel_thickness}"/>
             </geometry>
         </collision>
@@ -349,7 +374,7 @@
         </visual>
         <collision>
-            <origin xyz="${rocker_length/2} 0 ${rocker_height/2}"/>
-            <geometry>
-                <box size="${rocker_length} ${rocker_width} ${rocker_height}"/>
+             <origin xyz="0 0 -${tilted_link/2}" rpy="0 ${pi/2} 0"/>
+            <geometry>
+                <box size="${tilted_link} ${rocker_width} 0.025"/>
             </geometry>
         </collision>
@@ -374,5 +399,5 @@
         <collision>
             <geometry>
-                <sphere radius="${wheel_radius}"/>
+                <cylinder radius="${wheel_radius}" length="${wheel_thickness}"/>
             </geometry>
         </collision>
@@ -399,6 +424,6 @@
         </visual>
         <collision>
-            <geometry>
-                <sphere radius="${wheel_radius}"/>
+             <geometry>
+                <cylinder radius="${wheel_radius}" length="${wheel_thickness}"/>
             </geometry>
         </collision>

Commit message: Rename tilted_link to tilted_length in robot_core.xacro

File: play_ground/fred/auracle/description/robot_core.xacro (robot description, xacro)
@@ -10,5 +10,5 @@
     <xacro:property name="rocker_height" value="0.2"/>
      <xacro:property name="rocker_mass" value="0.2"/>
-    <xacro:property name="tilted_link" value="0.1"/>
+    <xacro:property name="tilted_length" value="0.1"/>
     <xacro:property name="tilted_mass" value="0.5"/>
     <xacro:property name="wheel_radius" value="0.033"/>
@@ -64,5 +64,5 @@
     </gazebo>
  <!-- DIFFERENTIAL LINK -->
-    <joint name="differential_link" type="continuous">
+    <joint name="differential_link_joint" type="continuous">
         <parent link="chassis"/>
         <child link="differential_link"/>
@@ -83,9 +83,9 @@
             </geometry>
         </collision>
-        <xacro:inertial_box mass="${tilted_mass}" x="${tilted_link}" y="${rocker_width}" z="${rocker_height}">
-            <origin xyz="${rocker_length/2} 0 ${rocker_height/2}" rpy="0 0 0"/>
-        </xacro:inertial_box>
-    </link>
-    !-- LEFT WHEEL ROCKER LINK -->
+        <xacro:inertial_box mass="${tilted_mass}" x="${tilted_length}" y="${rocker_width}" z="${rocker_height}">
+            <origin xyz="${rocker_length/2} 0 ${rocker_height/2}" rpy="0 0 0"/>
+        </xacro:inertial_box>
+    </link>
+    <!-- LEFT WHEEL ROCKER LINK -->
     <joint name="left_wheel_rocker_joint" type="fixed">
         <parent link="differential_link"/>
@@ -107,5 +107,5 @@
             </geometry>
         </collision>
-        <xacro:inertial_box mass="${tilted_mass}" x="${tilted_link}" y="${rocker_width}" z="${rocker_height}">
+        <xacro:inertial_box mass="${tilted_mass}" x="${tilted_length}" y="${rocker_width}" z="${rocker_height}">
             <origin xyz="${rocker_length/2} 0 ${rocker_height/2}" rpy="0 0 0"/>
         </xacro:inertial_box>
@@ -119,17 +119,17 @@
     <link name="tilted_link">
         <visual>
-            <origin xyz="0 0 -${tilted_link/2}" rpy="0 ${pi/2} 0"/>
-            <geometry>
-                <box size="${tilted_link} ${rocker_width} 0.025"/>
-            </geometry>
-            <material name="black"/>
-        </visual>
-        <collision>
-           <origin xyz="0 0 -${tilted_link/2}" rpy="0 ${pi/2} 0"/>
-            <geometry>
-                <box size="${tilted_link} ${rocker_width} 0.025"/>
-            </geometry>
-        </collision>
-        <xacro:inertial_box mass="${tilted_mass}" x="${tilted_link}" y="${rocker_width}" z="${rocker_height}">
+            <origin xyz="0 0 -${tilted_length/2}" rpy="0 ${pi/2} 0"/>
+            <geometry>
+                <box size="${tilted_length} ${rocker_width} 0.025"/>
+            </geometry>
+            <material name="black"/>
+        </visual>
+        <collision>
+           <origin xyz="0 0 -${tilted_length/2}" rpy="0 ${pi/2} 0"/>
+            <geometry>
+                <box size="${tilted_length} ${rocker_width} 0.025"/>
+            </geometry>
+        </collision>
+        <xacro:inertial_box mass="${tilted_mass}" x="${tilted_length}" y="${rocker_width}" z="${rocker_height}">
             <origin xyz="${rocker_length/2} 0 ${rocker_height/2}" rpy="0 0 0"/>
         </xacro:inertial_box>
@@ -143,17 +143,17 @@
     <link name="tilted_two_link">
         <visual>
-            <origin xyz="0 0 -${tilted_link/2}" rpy="0 ${pi/2} 0"/>
-            <geometry>
-                <box size="${tilted_link} ${rocker_width} 0.025"/>
-            </geometry>
-            <material name="black"/>
-        </visual>
-        <collision>
-           <origin xyz="0 0 -${tilted_link/2}" rpy="0 ${pi/2} 0"/>
-            <geometry>
-                <box size="${tilted_link} ${rocker_width} 0.025"/>
-            </geometry>
-        </collision>
-        <xacro:inertial_box mass="${tilted_mass}" x="${tilted_link}" y="${rocker_width}" z="${rocker_height}">
+            <origin xyz="0 0 -${tilted_length/2}" rpy="0 ${pi/2} 0"/>
+            <geometry>
+                <box size="${tilted_length} ${rocker_width} 0.025"/>
+            </geometry>
+            <material name="black"/>
+        </visual>
+        <collision>
+           <origin xyz="0 0 -${tilted_length/2}" rpy="0 ${pi/2} 0"/>
+            <geometry>
+                <box size="${tilted_length} ${rocker_width} 0.025"/>
+            </geometry>
+        </collision>
+        <xacro:inertial_box mass="${tilted_mass}" x="${tilted_length}" y="${rocker_width}" z="${rocker_height}">
             <origin xyz="${rocker_length/2} 0 ${rocker_height/2}" rpy="0 0 0"/>
         </xacro:inertial_box>
@@ -163,5 +163,5 @@
         <parent link="tilted_two_link"/>
         <child link="left_wheel_one"/>
-        <origin xyz="0 0 ${-tilted_link}" rpy="0 ${pi/2} 0" />
+        <origin xyz="0 0 -${tilted_length}" rpy="0 ${pi/2} 0" />
         <axis xyz="0 0 1"/>
     </joint>
@@ -193,18 +193,18 @@
     <link name="tilted_three_link">
         <visual>
-            <origin xyz="0 0 -${tilted_link/2}" rpy="0 ${pi/2} 0"/>
-            <geometry>
-                <box size="${tilted_link} ${rocker_width} 0.025"/>
-            </geometry>
-            <material name="black"/>
-        </visual>
-        <collision>
-            <origin xyz="0 0 -${tilted_link/2}" rpy="0 ${pi/2} 0"/>
-            <geometry>
-                <box size="${tilted_link} ${rocker_width} 0.025"/>
-            </geometry>
-        </collision>
-        <xacro:inertial_box mass="${tilted_mass}" x="${tilted_link}" y="${rocker_width}" z="${rocker_height}">
-            <origin xyz="${tilted_link/2} 0 ${rocker_height/2}" rpy="0 0 0"/>
+            <origin xyz="0 0 -${tilted_length/2}" rpy="0 ${pi/2} 0"/>
+            <geometry>
+                <box size="${tilted_length} ${rocker_width} 0.025"/>
+            </geometry>
+            <material name="black"/>
+        </visual>
+        <collision>
+            <origin xyz="0 0 -${tilted_length/2}" rpy="0 ${pi/2} 0"/>
+            <geometry>
+                <box size="${tilted_length} ${rocker_width} 0.025"/>
+            </geometry>
+        </collision>
+        <xacro:inertial_box mass="${tilted_mass}" x="${tilted_length}" y="${rocker_width}" z="${rocker_height}">
+            <origin xyz="${tilted_length/2} 0 ${rocker_height/2}" rpy="0 0 0"/>
         </xacro:inertial_box>
     </link>
@@ -213,5 +213,5 @@
         <parent link="tilted_three_link"/>
         <child link="left_wheel_three"/>
-        <origin xyz="0 0 ${-tilted_link}" rpy="0 ${pi/2} 0" />
+        <origin xyz="0 0 ${-tilted_length}" rpy="0 ${pi/2} 0" />
         <axis xyz="0 0 1"/>
     </joint>
@@ -239,5 +239,5 @@
         <parent link="tilted_link"/>
         <child link="left_wheel_two"/>
-        <origin xyz="0 0 ${-tilted_link}" rpy="0 ${pi/2} 0" />
+        <origin xyz="0 0 -${tilted_length}" rpy="0 ${pi/2} 0" />
         <axis xyz="0 0 1"/>
     </joint>
@@ -293,14 +293,14 @@
     <link name="tilted_link_two">
         <visual>
-            <origin xyz="0 0 -${tilted_link/2}" rpy="0 ${pi/2} 0"/>
-            <geometry>
-                <box size="${tilted_link} ${rocker_width} 0.025"/>
-            </geometry>
-            <material name="black"/>
-        </visual>
-        <collision>
-           <origin xyz="0 0 -${tilted_link/2}" rpy="0 ${pi/2} 0"/>
-            <geometry>
-                <box size="${tilted_link} ${rocker_width} 0.025"/>
+            <origin xyz="0 0 -${tilted_length/2}" rpy="0 ${pi/2} 0"/>
+            <geometry>
+                <box size="${tilted_length} ${rocker_width} 0.025"/>
+            </geometry>
+            <material name="black"/>
+        </visual>
+        <collision>
+           <origin xyz="0 0 -${tilted_length/2}" rpy="0 ${pi/2} 0"/>
+            <geometry>
+                <box size="${tilted_length} ${rocker_width} 0.025"/>
             </geometry>
         </collision>
@@ -317,14 +317,14 @@
     <link name="tilted_two_link_two">
         <visual>
-            <origin xyz="0 0 -${tilted_link/2}" rpy="0 ${pi/2} 0"/>
-            <geometry>
-                <box size="${tilted_link} ${rocker_width} 0.025"/>
-            </geometry>
-            <material name="black"/>
-        </visual>
-        <collision>
-           <origin xyz="0 0 -${tilted_link/2}" rpy="0 ${pi/2} 0"/>
-            <geometry>
-                <box size="${tilted_link} ${rocker_width} 0.025"/>
+            <origin xyz="0 0 -${tilted_length/2}" rpy="0 ${pi/2} 0"/>
+            <geometry>
+                <box size="${tilted_length} ${rocker_width} 0.025"/>
+            </geometry>
+            <material name="black"/>
+        </visual>
+        <collision>
+           <origin xyz="0 0 -${tilted_length/2}" rpy="0 ${pi/2} 0"/>
+            <geometry>
+                <box size="${tilted_length} ${rocker_width} 0.025"/>
             </geometry>
         </collision>
@@ -337,5 +337,5 @@
         <parent link="tilted_two_link_two"/>
         <child link="right_wheel_one"/>
-        <origin xyz="0 0 ${-tilted_link}" rpy="0 ${pi/2} 0" />
+        <origin xyz="0 0 ${-tilted_length}" rpy="0 ${pi/2} 0" />
         <axis xyz="0 0 1"/>
     </joint>
@@ -367,14 +367,14 @@
     <link name="tilted_two_link_three">
         <visual>
-            <origin xyz="0 0 -${tilted_link/2}" rpy="0 ${pi/2} 0"/>
-            <geometry>
-                <box size="${tilted_link} ${rocker_width} 0.025"/>
-            </geometry>
-            <material name="black"/>
-        </visual>
-        <collision>
-             <origin xyz="0 0 -${tilted_link/2}" rpy="0 ${pi/2} 0"/>
-            <geometry>
-                <box size="${tilted_link} ${rocker_width} 0.025"/>
+            <origin xyz="0 0 -${tilted_length/2}" rpy="0 ${pi/2} 0"/>
+            <geometry>
+                <box size="${tilted_length} ${rocker_width} 0.025"/>
+            </geometry>
+            <material name="black"/>
+        </visual>
+        <collision>
+             <origin xyz="0 0 -${tilted_length/2}" rpy="0 ${pi/2} 0"/>
+            <geometry>
+                <box size="${tilted_length} ${rocker_width} 0.025"/>
             </geometry>
         </collision>
@@ -387,5 +387,5 @@
         <parent link="tilted_two_link_three"/>
         <child link="right_wheel_three"/>
-        <origin xyz="0 0 ${-tilted_link}" rpy="0 ${pi/2} 0" />
+        <origin xyz="0 0 ${-tilted_length}" rpy="0 ${pi/2} 0" />
         <axis xyz="0 0 1"/>
     </joint>
@@ -413,5 +413,5 @@
         <parent link="tilted_link_two"/>
         <child link="right_wheel_two"/>
-        <origin xyz="0 0 ${-tilted_link}" rpy="0 ${pi/2} 0" />
+        <origin xyz="0 0 ${-tilted_length}" rpy="0 ${pi/2} 0" />
         <axis xyz="0 0 1"/>
     </joint>
