Commit message: Adjust laser_joint origin position in lidar.xacro

File: play_ground/fred/auracle/description/lidar.xacro (robot description, xacro)
@@ -4,5 +4,5 @@
         <parent link="chassis"/>
         <child link="laser_frame"/>
-        <origin xyz="0.2 0 0.085" rpy="0 0 0"/>
+        <origin xyz="0.15 0 0.085" rpy="0 0 0"/>
     </joint>
     <link name="laser_frame">
