Commit message: RDI-789: add slam_toolbos

File: robot_software/robot_2_ws/src/robot_2_description/urdf/robot_2.urdf.xacro (robot description, xacro)
@@ -1,8 +1,16 @@
 <?xml version="1.0"?>
 <robot xmlns:xacro="http://www.ros.org/wiki/xacro" name="robot_2">
-    <!-- Relative paths remain identical since files live in the same directory -->
-    <xacro:include filename="robot_core.xacro" />
-    <xacro:include filename="gazebo_control.xacro" />
-    <!-- <xacro:include filename="ros2_control.xacro" /> -->
-    <xacro:include filename="lidar.xacro" />
+    <!-- Select whether to use ros2_control or Gazebo DiffDrive -->
+    <xacro:arg name="use_ros2_control" default="true"/>
+    <!-- Robot model -->
+    <xacro:include filename="robot_core.xacro"/>
+    <!-- Select control backend -->
+    <xacro:if value="$(arg use_ros2_control)">
+        <xacro:include filename="ros2_control.xacro"/>
+    </xacro:if>
+    <xacro:unless value="$(arg use_ros2_control)">
+        <xacro:include filename="gazebo_control.xacro"/>
+    </xacro:unless>
+    <!-- Sensors -->
+    <xacro:include filename="lidar.xacro"/>
 </robot>

File: robot_software/robot_2_ws/src/robot_2_description/urdf/robot_core.xacro (robot description, xacro)
@@ -11,6 +11,20 @@
         <color rgba="0 0 0 1"/>
     </material>
+    <material name="red">
+        <color rgba="1 0 0 1"/>
+    </material>
+    <material name="purple">
+        <color rgba="0.5 0 0.5 1"/>
+    </material>
     <link name="base_link">
     </link>
+    <link name="base_footprint">
+    </link>
+    <joint name="base_footprint_joint" type="fixed">
+        <parent link="base_footprint"/>
+        <child link="base_link"/>
+        <!-- Offset matches your wheel radius exactly so base_footprint rests flat on the floor -->
+        <origin xyz="0 0 -0.0425" rpy="0 0 0"/>
+    </joint>
     <!-- CHASSIS -->
     <joint name="chassis_joint" type="fixed">
