Commit message: RDI-78: add object in gamefield

File: robot_software/robot_2_ws/src/robot_2_description/urdf/robot_core.xacro (robot description, xacro)
@@ -24,6 +24,6 @@
         <parent link="base_footprint"/>
         <child link="base_link"/>
-        <!-- Offset matches your wheel radius exactly so base_footprint rests flat on the floor -->
-        <origin xyz="0 0 -0.0425" rpy="0 0 0"/>
+        <!-- FIX: Offset changed to positive so base_link is elevated properly above floor grid -->
+        <origin xyz="0 0 0.0425" rpy="0 0 0"/>
     </joint>
     <!-- CHASSIS -->
@@ -39,5 +39,5 @@
                 <box size="0.3 0.25 0.18"/>
             </geometry>
-            <material name="white"/>
+            <material name="purple"/>
         </visual>
         <collision>

File: robot_software/robot_2_ws/src/robot_2_description/urdf/ros2_control.xacro (robot description, xacro)
@@ -29,8 +29,10 @@
   <!-- Gazebo ros2_control plugin -->
   <gazebo>
-    <plugin
-      filename="gz_ros2_control-system"
-      name="gz_ros2_control::GazeboSimSystem">
+    <plugin filename="gz_ros2_control-system" name="gz_ros2_control::GazeboSimROS2ControlPlugin">
       <parameters>$(find robot_2_bringup)/config/my_controllers.yaml</parameters>
+      <!-- FIX: Explicitly namespace the internal controller manager plugin instance -->
+      <ros>
+        <namespace>/robot_2</namespace>
+      </ros>
     </plugin>
   </gazebo>
