Commit message: RDI-78: Update laser joint origin position in lidar.xacro

File: robot_software/robot_2_ws/src/robot_2_description/urdf/lidar.xacro (robot description, xacro)
@@ -4,5 +4,5 @@
     <parent link="chassis"/>
     <child link="laser_frame"/>
-    <origin xyz="0.09 0 0.19" rpy="0 0 0"/>
+    <origin xyz="0.15 0 0.19" rpy="0 0 0"/>
   </joint>
   <link name="laser_frame">
