Commit message: RDI - 89: Add ROS2 control interface for Arduino and Gazebo simulation

File: robot_software/robot_2_ws/src/robot_2_description/urdf/ros2_control.xacro (robot description, xacro)
@@ -1,39 +1,105 @@
 <?xml version="1.0"?>
 <robot xmlns:xacro="http://ros.org">
-  <!-- ros2_control hardware definition -->
-  <ros2_control name="GazeboSimSystem" type="system">
-    <hardware>
-      <plugin>gz_ros2_control/GazeboSimSystem</plugin>
-    </hardware>
-    <joint name="front_left_wheel_joint">
-      <command_interface name="velocity"/>
-      <state_interface name="position"/>
-      <state_interface name="velocity"/>
-    </joint>
-    <joint name="front_right_wheel_joint">
-      <command_interface name="velocity"/>
-      <state_interface name="position"/>
-      <state_interface name="velocity"/>
-    </joint>
-    <joint name="back_left_wheel_joint">
-      <command_interface name="velocity"/>
-      <state_interface name="position"/>
-      <state_interface name="velocity"/>
-    </joint>
-    <joint name="back_right_wheel_joint">
-      <command_interface name="velocity"/>
-      <state_interface name="position"/>
-      <state_interface name="velocity"/>
-    </joint>
-  </ros2_control>
-  <!-- Gazebo ros2_control plugin -->
-  <gazebo>
-    <plugin filename="gz_ros2_control-system" name="gz_ros2_control::GazeboSimROS2ControlPlugin">
-      <parameters>$(find robot_2_bringup)/config/my_controllers.yaml</parameters>
-      <ros>
-        <namespace>/robot_2</namespace>
-      </ros>
-      <robot_param_node>/robot_2/robot_state_publisher</robot_param_node>
-    </plugin>
-  </gazebo>
+  <!--
+    Select Gazebo simulation hardware vs the real Arduino/L298 robot.
+    Defaults to sim (false = not real) to preserve existing behaviour
+    for anyone launching without passing this explicitly - forwarded
+    from robot_state_publisher.launch.py via xacro mappings.
+  -->
+  <xacro:arg name="sim_mode" default="false"/>
+  <!-- ====================================================== -->
+  <!-- SIMULATION            -->
+  <!-- ====================================================== -->
+  <xacro:if value="$(arg sim_mode)">
+    <!-- ros2_control hardware definition -->
+    <ros2_control name="GazeboSimSystem" type="system">
+      <hardware>
+        <plugin>gz_ros2_control/GazeboSimSystem</plugin>
+      </hardware>
+      <joint name="front_left_wheel_joint">
+        <command_interface name="velocity"/>
+        <state_interface name="position"/>
+        <state_interface name="velocity"/>
+      </joint>
+      <joint name="front_right_wheel_joint">
+        <command_interface name="velocity"/>
+        <state_interface name="position"/>
+        <state_interface name="velocity"/>
+      </joint>
+      <joint name="back_left_wheel_joint">
+        <command_interface name="velocity"/>
+        <state_interface name="position"/>
+        <state_interface name="velocity"/>
+      </joint>
+      <joint name="back_right_wheel_joint">
+        <command_interface name="velocity"/>
+        <state_interface name="position"/>
+        <state_interface name="velocity"/>
+      </joint>
+    </ros2_control>
+    <!-- Gazebo ros2_control plugin -->
+    <gazebo>
+      <plugin filename="gz_ros2_control-system" name="gz_ros2_control::GazeboSimROS2ControlPlugin">
+        <parameters>$(find robot_2_bringup)/config/my_controllers.yaml</parameters>
+        <ros>
+          <namespace>/robot_2</namespace>
+        </ros>
+        <robot_param_node>/robot_2/robot_state_publisher</robot_param_node>
+      </plugin>
+    </gazebo>
+  </xacro:if>
+  <!-- ====================================================== -->
+  <!-- REAL ROBOT (Arduino Uno + 2x L298N + quadrature enc.)   -->
+  <!-- ====================================================== -->
+  <xacro:unless value="$(arg sim_mode)">
+    <ros2_control name="RealRobotSystem" type="system">
+      <hardware>
+        <plugin>robot_2_hardware/Robot2System</plugin>
+        <!-- Arduino serial configuration -->
+        <param name="device">/dev/ttyUSB_ARDUINO</param>
+        <param name="baud_rate">57600</param>
+        <param name="timeout_ms">100</param>
+        <!-- Encoder configuration -->
+        <param name="encoder_ticks_per_rev">1980</param>
+        <!--
+          Arduino PID period, in SECONDS. on_init() reads a parameter
+          named exactly "pid_period" (see getNumericParameter calls in
+          robot_2_system.cpp) - NOT "pid_period_ms". 0.05s = 50ms,
+          matching the firmware's config.h PID_PERIOD.
+        -->
+        <param name="pid_period">0.05</param>
+        <!-- Wheel geometry -->
+        <param name="wheel_radius">0.0425</param>
+      </hardware>
+      <!--
+        Joint order below MUST match the index assumption hard-coded
+        in Robot2System::write()/read():
+          0 = front_left, 1 = front_right, 2 = back_left, 3 = back_right
+      -->
+      <!-- LEFT FRONT (index 0) -->
+      <joint name="front_left_wheel_joint">
+        <command_interface name="velocity"/>
+        <state_interface name="position"/>
+        <state_interface name="velocity"/>
+      </joint>
+      <!-- RIGHT FRONT (index 1) -->
+      <joint name="front_right_wheel_joint">
+        <command_interface name="velocity"/>
+        <state_interface name="position"/>
+        <state_interface name="velocity"/>
+      </joint>
+      <!-- LEFT REAR (index 2) -->
+      <joint name="back_left_wheel_joint">
+        <command_interface name="velocity"/>
+        <state_interface name="position"/>
+        <state_interface name="velocity"/>
+      </joint>
+      <!-- RIGHT REAR (index 3) -->
+      <joint name="back_right_wheel_joint">
+        <command_interface name="velocity"/>
+        <state_interface name="position"/>
+        <state_interface name="velocity"/>
+      </joint>
+    </ros2_control>
+  </xacro:unless>
 </robot>
