Commit message: Fix robot URDF file to stop tilting

File: play_ground/emmanuel/auracle/description/robot_core.xacro (robot description, xacro)
@@ -64,5 +64,5 @@
     </gazebo>
  <!-- LEFT WHEEL ROCKER LINK -->
-    <joint name="left_wheel_rocker_joint" type="continuous">
+    <joint name="left_wheel_rocker_joint" type="fixed">
         <parent link="base_link"/>
         <child link="left_rocker"/>
@@ -78,7 +78,7 @@
         </visual>
         <collision>
-            <origin xyz="${rocker_length/2} 0 ${rocker_height/2}"/>
-            <geometry>
-                <box size="${rocker_length} ${rocker_width} ${rocker_height}"/>
+            <origin xyz="0 0 0" rpy="0 0 ${-pi/2}"/>
+            <geometry>
+                <box size="${rocker_length} ${rocker_width} 0.025"/>
             </geometry>
         </collision>
@@ -102,7 +102,7 @@
         </visual>
         <collision>
-            <origin xyz="${rocker_length/2} 0 ${rocker_height/2}"/>
-            <geometry>
-                <box size="${rocker_length} ${rocker_width} ${rocker_height}"/>
+            <origin xyz="0 0 -${tilted_link/2}" rpy="0 ${pi/2} 0"/>
+            <geometry>
+                <box size="${tilted_link} ${rocker_width} 0.025"/>
             </geometry>
         </collision>
@@ -112,5 +112,5 @@
     </link>
         <!-- TILTED LINK2 -->
-    <joint name="tilted_two_joint" type="fixed">
+    <joint name="tilted_two_joint" type="continuous">
         <parent link="left_rocker"/>
         <child link="tilted_two_link"/>
@@ -165,7 +165,7 @@
     <!-- TILTED LINK6 -->
     <joint name="tilted_three_joint" type="fixed">
-        <parent link="left_rocker"/>
+        <parent link="tilted_two_link"/>
         <child link="tilted_three_link"/>
-        <origin xyz="0 ${-rocker_length/2} 0" rpy="${pi/4} 0 0" />
+        <origin xyz="0 0 0" rpy="${pi/2} 0 0" />
     </joint>
     <link name="tilted_three_link">
@@ -178,7 +178,7 @@
         </visual>
         <collision>
-            <origin xyz="${rocker_length/2} 0 ${rocker_height/2}"/>
-            <geometry>
-                <box size="${rocker_length} ${rocker_width} ${rocker_height}"/>
+            <origin xyz="0 0 -${tilted_link/2}" rpy="0 ${pi/2} 0"/>
+            <geometry>
+                <box size="${tilted_link} ${rocker_width} 0.025"/>
             </geometry>
         </collision>
@@ -240,5 +240,5 @@
     </gazebo>
     <!-- RIGHT WHEEL ROCKER LINK -->
-    <joint name="right_wheel_rocker_joint" type="continuous">
+    <joint name="right_wheel_rocker_joint" type="fixed">
         <parent link="base_link"/>
         <child link="right_rocker"/>
@@ -254,7 +254,7 @@
         </visual>
         <collision>
-            <origin xyz="${rocker_length/2} 0 ${rocker_height/2}"/>
-            <geometry>
-                <box size="${rocker_length} ${rocker_width} ${rocker_height}"/>
+            <origin xyz="0 0 0" rpy="0 0 ${-pi/2}"/>
+            <geometry>
+                <box size="${rocker_length} ${rocker_width} 0.025"/>
             </geometry>
         </collision>
@@ -278,7 +278,7 @@
         </visual>
         <collision>
-            <origin xyz="${rocker_length/2} 0 ${rocker_height/2}"/>
-            <geometry>
-                <box size="${rocker_length} ${rocker_width} ${rocker_height}"/>
+            <origin xyz="0 0 -${tilted_link/2}" rpy="0 ${pi/2} 0"/>
+            <geometry>
+                <box size="${tilted_link} ${rocker_width} 0.025"/>
             </geometry>
         </collision>
@@ -288,5 +288,5 @@
     </link>
     <!-- TILTED LINK2 -->
-    <joint name="tilted_two_joint_two" type="fixed">
+    <joint name="tilted_two_joint_two" type="continuous">
         <parent link="right_rocker"/>
         <child link="tilted_two_link_two"/>
@@ -302,7 +302,7 @@
         </visual>
         <collision>
-            <origin xyz="${rocker_length/2} 0 ${rocker_height/2}"/>
-            <geometry>
-                <box size="${rocker_length} ${rocker_width} ${rocker_height}"/>
+            <origin xyz="0 0 -${tilted_link/2}" rpy="0 ${pi/2} 0"/>
+            <geometry>
+                <box size="${tilted_link} ${rocker_width} 0.025"/>
             </geometry>
         </collision>
@@ -339,7 +339,7 @@
     <!-- TILTED LINK3 -->
      <joint name="tilted_two_joint_three" type="fixed">
-        <parent link="right_rocker"/>
+        <parent link="tilted_two_link_two"/>
         <child link="tilted_two_link_three"/>
-        <origin xyz="0 ${-rocker_length/2} 0" rpy="${pi/4} 0 0" />
+        <origin xyz="0 0 0" rpy="${pi/2} 0 0" />
     </joint>
     <link name="tilted_two_link_three">
@@ -352,7 +352,7 @@
         </visual>
         <collision>
-            <origin xyz="${rocker_length/2} 0 ${rocker_height/2}"/>
-            <geometry>
-                <box size="${rocker_length} ${rocker_width} ${rocker_height}"/>
+            <origin xyz="0 0 -${tilted_link/2}" rpy="0 ${pi/2} 0"/>
+            <geometry>
+                <box size="${tilted_link} ${rocker_width} 0.025"/>
             </geometry>
         </collision>
